Commit message: Created Map :)

File: urdf/robot.xacro (robot description, xacro)
@@ -10,7 +10,6 @@
     <xacro:chasis />
     <!-- Robot Wheels -->
-    <xacro:wheel side="right" position="front" offset_x="${chasis_length/2 - 0.1}" offset_y="${-(chasis_width/2 + 0.05)}" />
-    <xacro:wheel side="left" position="front" offset_x="${chasis_length/2 - 0.1}" offset_y="${chasis_width/2 + 0.05}" />
-    <xacro:wheel side="right" position="back" offset_x="${-(chasis_length/2 - 0.1)}" offset_y="${-(chasis_width/2 + 0.05)}" />
-    <xacro:wheel side="left" position="back" offset_x="${-(chasis_length/2 - 0.1)}" offset_y="${chasis_width/2 + 0.05}" />
+    <xacro:wheel prefix="left" y_offset="${chasis_radius}" />
+    <xacro:wheel prefix="right" y_offset="${-(chasis_radius)}" />
+    <xacro:passive_wheel x_offset="0.065" z_offset="-0.02" />
 </robot>

File: urdf/xacro/chasis.xacro (robot description, xacro)
@@ -1,37 +1,37 @@
 <?xml version="1.0"?>
 <robot xmlns:xacro="http://www.ros.org/wiki/xacro">
-    <xacro:property name="head_mass" value="0.1" />
-    <xacro:property name="head_radius" value="0.2" />
-    <xacro:property name="head_inertia_calc" value="${(2/5) * head_mass * (head_radius * head_radius)}" />
-    <xacro:property name="chasis_mass" value="0.2" />
-    <xacro:property name="chasis_width" value="0.8" />
-    <xacro:property name="chasis_height" value="0.25" />
-    <xacro:property name="chasis_length" value="1" />
-    <xacro:property name="chasis_inertia_calc_ixx" value="${(1/12) * chasis_mass * ((chasis_height * chasis_height) + (chasis_length * chasis_length))}" />
-    <xacro:property name="chasis_inertia_calc_iyy" value="${(1/12) * chasis_mass * ((chasis_width * chasis_width) + (chasis_height * chasis_height))}" />
-    <xacro:property name="chasis_inertia_calc_izz" value="${(1/12) * chasis_mass * ((chasis_width * chasis_width) + (chasis_length * chasis_length))}" />
+    <xacro:property name="head_mass" value="0.02" />
+    <xacro:property name="head_width" value="0.03" />
+    <xacro:property name="head_length" value="0.03" />
+    <xacro:property name="head_height" value="0.03" />
+    <xacro:property name="head_inertia_calc_ixx" value="${(1/12) * head_mass * ((head_height * head_height) + (head_length * head_length))}" />
+    <xacro:property name="head_inertia_calc_iyy" value="${(1/12) * head_mass * ((head_width * head_width) + (head_height * head_height))}" />
+    <xacro:property name="head_inertia_calc_izz" value="${(1/12) * head_mass * ((head_width * head_width) + (head_length * head_length))}" />
+    <xacro:property name="chasis_mass" value="0.1" />
+    <xacro:property name="chasis_radius" value="0.0825" />
+    <xacro:property name="chasis_height" value="0.025" />
+    <xacro:property name="chasis_inertia_calc" value="${(1/12) * chasis_mass * ((3 * (chasis_radius * chasis_radius)) + (chasis_height * chasis_height))}" />
+    <xacro:property name="chasis_inertia_calc_izz" value="${(1/2) * chasis_mass * (chasis_radius * chasis_radius)}" />
     <xacro:macro name="chasis">
         <!-- Robot Head -->
         <link name="head">
             <visual>
-                <origin xyz="0 0 0" rpy="0.0 0.0 0.0" />
                 <geometry>
-                    <sphere radius="${head_radius}" />
+                    <box size="${head_length} ${head_width} ${head_height}" />
                 </geometry>
                 <material name="red" />
             </visual>
             <collision>
-                <origin xyz="0 0 0" rpy="0.0 0.0 0.0" />
                 <geometry>
-                    <sphere radius="${head_radius}" />
+                    <box size="${head_length} ${head_width} ${head_height}" />
                 </geometry>
             </collision>
             <inertial>
                 <mass value="${chasis_mass}"/>
-                <inertia ixx="${head_inertia_calc}" ixy="0.0" ixz="0.0" iyy="${head_inertia_calc}" iyz="0.0" izz="${head_inertia_calc}"/>
+                <inertia ixx="${head_inertia_calc_ixx}" ixy="0.0" ixz="0.0" iyy="${head_inertia_calc_iyy}" iyz="0.0" izz="${head_inertia_calc_izz}"/>
             </inertial>
         </link>
         <joint name="joint_chasis__head" type="fixed">
-            <origin xyz="0.25 0 0.15" rpy="0.0 0.0 0.0" />
+            <origin xyz="0.065 0 0.025" rpy="0 0 0" />
             <parent link="chasis"/>
             <child link="head"/>
@@ -40,19 +40,17 @@
         <link name="chasis">
             <visual>
-                <origin xyz="0.0 0.0 0.0" rpy="0.0 0.0 0.0" />
                 <geometry>
-                    <box size="${chasis_length} ${chasis_width} ${chasis_height}" />
+                    <cylinder radius="${chasis_radius}" length="${chasis_height}" />
                 </geometry>
                 <material name="red" />
             </visual>
             <collision>
-                <origin xyz="0.0 0.0 0.0" rpy="0.0 0.0 0.0" />
                 <geometry>
-                    <box size="${chasis_length} ${chasis_width} ${chasis_height}" />
+                    <cylinder radius="${chasis_radius}" length="${chasis_height}" />
                 </geometry>
             </collision>
             <inertial>
                 <mass value="${chasis_mass}"/>
-                <inertia ixx="${chasis_inertia_calc_ixx}" ixy="0.0" ixz="0.0" iyy="${chasis_inertia_calc_iyy}" iyz="0.0" izz="${chasis_inertia_calc_izz}"/>
+                <inertia ixx="${chasis_inertia_calc}" ixy="0.0" ixz="0.0" iyy="${chasis_inertia_calc}" iyz="0.0" izz="${chasis_inertia_calc_izz}"/>
             </inertial>
         </link>

File: urdf/xacro/gazebo.xacro (robot description, xacro)
@@ -1,7 +1,8 @@
 <?xml version="1.0"?>
 <robot xmlns:xacro="http://www.ros.org/wiki/xacro">
-    <xacro:macro name="robot_dynamics" params="mu1 mu2">
-        <mu1 value="${mu1}" />
-        <mu2 value="${mu2}" />
+    <xacro:include filename="$(find ceerii_mobile_bot)/urdf/xacro/sensors.xacro"/>
+    <xacro:macro name="wheel_dynamics">
+        <mu1 value="200.0"/>
+        <mu2 value="100.0"/>
         <kp value="10000000.0" />
         <kd value="1.0" />
@@ -13,20 +14,21 @@
     <gazebo reference="head">
         <material>Gazebo/Red</material>
+        <xacro:laser_sensor />
     </gazebo>
-    <gazebo reference="right_front_wheel">
-        <xacro:robot_dynamics mu1="200" mu2="100" />
+    <gazebo reference="passive_wheel_holder">
         <material>Gazebo/Black</material>
     </gazebo>
-    <gazebo reference="right_back_wheel">
-        <xacro:robot_dynamics mu1="200" mu2="100" />
+    <gazebo reference="passive_wheel">
+        <mu1 value="0"/>
+        <mu2 value="0"/>
         <material>Gazebo/Black</material>
     </gazebo>
-    <gazebo reference="left_front_wheel">
-        <xacro:robot_dynamics mu1="200" mu2="100" />
+    <gazebo reference="left_wheel">
         <material>Gazebo/Black</material>
+        <xacro:wheel_dynamics />
     </gazebo>
-    <gazebo reference="left_back_wheel">
-        <xacro:robot_dynamics mu1="200" mu2="100" />
+    <gazebo reference="right_wheel">
         <material>Gazebo/Black</material>
+        <xacro:wheel_dynamics />
     </gazebo>
     <!-- General Gazebo Plugins -->

File: urdf/xacro/wheels.xacro (robot description, xacro)
@@ -3,21 +3,29 @@
     <xacro:include filename="$(find ceerii_mobile_bot)/urdf/xacro/transmissions.xacro"/>
     <xacro:property name="wheel_mass" value="0.015" />
-    <xacro:property name="wheel_radius" value="0.2" />
-    <xacro:property name="wheel_height" value="0.1" />
+    <xacro:property name="wheel_radius" value="0.035" />
+    <xacro:property name="wheel_height" value="0.008" />
+    <xacro:property name="passive_wheel_mass" value="0.02" />
+    <xacro:property name="passive_wheel_radius" value="0.01" />
+    <xacro:property name="passive_wheel_holder_mass" value="0.02" />
+    <xacro:property name="passive_wheel_holder_radius" value="0.01" />
+    <xacro:property name="passive_wheel_holder_height" value="0.018" />
+    <xacro:property name="passive_wheel_inertia_calc" value="${(2/5) * passive_wheel_mass * (passive_wheel_radius * passive_wheel_radius)}" />
+    <xacro:property name="wheel_inertia_calc_izz" value="${(1/2) * wheel_mass * (wheel_radius * wheel_radius)}" />
     <xacro:property name="wheel_inertia_calc" value="${(1/12) * wheel_mass * ((3 * (wheel_radius * wheel_radius)) + (wheel_height * wheel_height))}" />
-    <xacro:property name="wheel_inertia_calc_izz" value="${(1/2) * wheel_mass * (wheel_radius * wheel_radius)}" />
-    <xacro:macro name="wheel" params="side position offset_x offset_y">
-        <link name="${side}_${position}_wheel">
+    <xacro:property name="passive_wheel_holder_inertia_calc_izz" value="${(1/2) * passive_wheel_holder_mass * (passive_wheel_holder_radius * passive_wheel_holder_radius)}" />
+    <xacro:property name="passive_wheel_holder_inertia_calc" value="${(1/12) * passive_wheel_holder_mass * ((3 * (passive_wheel_holder_radius * passive_wheel_holder_radius)) + (passive_wheel_holder_height * passive_wheel_holder_height))}" />
+    <xacro:macro name="wheel" params="prefix y_offset">
+        <link name="${prefix}_wheel">
             <visual>
-                <origin xyz="0 0 0" rpy="${pi/2} 0 0"/>
+                <origin xyz="0 0 0" rpy="${pi/2} 0 0" />
                 <geometry>
-                    <cylinder radius="${wheel_radius}" length="${wheel_height}"/>
+                    <cylinder radius="${wheel_radius}" length="${wheel_height}" />
                 </geometry>
-                <material name="black"/>
+                <material name="black" />
             </visual>
             <collision>
-                <origin xyz="0 0 0" rpy="${pi/2} 0 0"/>
+                <origin xyz="0 0 0" rpy="${pi/2} 0 0" />
                 <geometry>
-                    <cylinder radius="${wheel_radius}" length="${wheel_height}"/>
+                    <cylinder radius="${wheel_radius}" length="${wheel_height}" />
                 </geometry>
             </collision>
@@ -27,12 +35,60 @@
             </inertial>
         </link>
-        <joint name="joint_${side}_${position}_wheel" type="continuous">
+        <joint name="joint_chasis__${prefix}_wheel" type="continuous">
             <parent link="chasis"/>
-            <child link="${side}_${position}_wheel"/>
-            <origin xyz="${offset_x} ${offset_y} 0.0" rpy="0.0 0.0 0.0"/>
-            <axis xyz="0.0 1 0.0"/>
+            <child link="${prefix}_wheel"/>
+            <origin xyz="0 ${y_offset} 0" rpy="0 0 0" />
+            <axis xyz="0 1 0"/>
         </joint>
         <!-- Robot Joints' Transmission -->
-        <xacro:wheel_transmission wheelJointName="joint_${side}_${position}_wheel"  />
+        <xacro:wheel_transmission wheelJointName="joint_chasis__${prefix}_wheel"  />
+    </xacro:macro>
+    <xacro:macro name="passive_wheel" params="z_offset x_offset">
+        <link name="passive_wheel_holder">
+            <visual>
+                <origin xyz="0 0 ${z_offset}" />
+                <geometry>
+                    <cylinder radius="${passive_wheel_holder_radius}" length="${passive_wheel_holder_height}" />
+                </geometry>
+                <material name="black"></material>
+            </visual>
+            <collision>
+                <origin xyz="0 0 ${z_offset}" />
+                <geometry>
+                    <cylinder radius="${passive_wheel_holder_radius}" length="${passive_wheel_holder_height}" />
+                </geometry>
+            </collision>
+            <inertial>
+                <mass value="${passive_wheel_holder_mass}"/>
+                <inertia ixx="${passive_wheel_holder_inertia_calc}" ixy="0.0" ixz="0.0" iyy="${passive_wheel_holder_inertia_calc}" iyz="0.0" izz="${passive_wheel_holder_inertia_calc_izz}"/>
+            </inertial>
+        </link>
+        <joint name="joint_chasis__passive_wheel_holder" type="fixed">
+            <origin xyz="${x_offset} 0 0" rpy="0 0 0" />
+            <parent link="chasis"/>
+            <child link="passive_wheel_holder"/>
+        </joint>
+        <link name="passive_wheel">
+            <visual>
+                <geometry>
+                    <sphere radius="${passive_wheel_radius}" />
+                </geometry>
+                <material name="black"></material>
+            </visual>
+            <collision>
+                <geometry>
+                    <sphere radius="${passive_wheel_radius}" />
+                </geometry>
+            </collision>
+            <inertial>
+                <mass value="${passive_wheel_mass}"/>
+                 <inertia ixx="${passive_wheel_inertia_calc}" ixy="0.0" ixz="0.0" iyy="${passive_wheel_inertia_calc}" iyz="0.0" izz="${passive_wheel_inertia_calc}"/>
+            </inertial>
+        </link>
+        <joint name="joint_passive_wheel_holder__passive_wheel" type="fixed">
+            <origin xyz="0 0 ${z_offset - 0.005}" rpy="0 0 0" />
+            <parent link="passive_wheel_holder"/>
+            <child link="passive_wheel"/>
+        </joint>
     </xacro:macro>
 </robot>
